File: motor_drive_REV_1/ADA4571WHRZ.sch (KiCad schematic (older format))
At the start: 2 parts

Commit message: organizing pinout and BOM
Parts:
- C14: renamed from C?; footprint (none) -> motor_drive_footprints:C_0603_1608Metric
- U5: renamed from U?; footprint R_8 -> motor_drive_footprints:AD8418ABRMZ-RL
Connections:
- net VDD: now also C14.1
Changed lines of the file:
@@
 $Descr A4 11693 8268
 encoding utf-8
-Sheet 13 14
+Sheet 10 14
 Title ""
 Date ""
@@
 $EndDescr
 $Comp
-L motor_drive:ADA4571WHRZ-R7 U?
+L motor_drive:ADA4571WHRZ-R7 U5
 U 1 1 5E373274
 P 4450 3850
-F 0 "U?" H 5250 4237 60  0000 C CNN
+F 0 "U5" H 5250 4237 60  0000 C CNN
 F 1 "ADA4571WHRZ-R7" H 5250 4131 60  0000 C CNN
-F 2 "R_8" H 5250 4090 60  0001 C CNN
+F 2 "motor_drive_footprints:AD8418ABRMZ-RL" H 5250 4090 60  0001 C CNN
 F 3 "" H 4450 3850 60  0000 C CNN
 	1    4450 3850
@@
 	6200 4050 6200 4450
 Wire Wire Line
-	4450 4150 3550 4150
-Wire Wire Line
 	3550 4150 3550 4850
 Wire Wire Line
@@
 NoConn ~ 4450 4050
 Wire Wire Line
-	3400 3850 4450 3850
+	4450 4150 3550 4150
 $Comp
-L motor_drive:C C?
+L motor_drive:C C14
 U 1 1 5E374B8C
 P 3550 4000
-F 0 "C?" V 3298 4000 50  0000 C CNN
+F 0 "C14" V 3298 4000 50  0000 C CNN
 F 1 "C" V 3389 4000 50  0000 C CNN
-F 2 "" H 3588 3850 50  0001 C CNN
+F 2 "motor_drive_footprints:C_0603_1608Metric" H 3588 3850 50  0001 C CNN
 F 3 "~" H 3550 4000 50  0001 C CNN
 	1    3550 4000
 	1    0    0    -1
 $EndComp
+Wire Wire Line
+	4450 3850 3550 3850
+Wire Wire Line
+	3550 3850 3400 3850
+Connection ~ 3550 3850
 $EndSCHEMATC

Commit message: working on adding thermistors but encountered too many hierarchicaly copies bug
Parts:
- added C13: 0.01uF, motor_drive_footprints:C_0603_1608Metric, symbol motor_drive:C
- C12: renamed from C14; value C -> 2.2uF
Changed lines of the file:
@@
 	4450 4150 3550 4150
 $Comp
-L motor_drive:C C14
+L motor_drive:C C12
 U 1 1 5E374B8C
 P 3550 4000
-F 0 "C14" V 3298 4000 50  0000 C CNN
-F 1 "C" V 3389 4000 50  0000 C CNN
+F 0 "C12" V 3298 4000 50  0000 C CNN
+F 1 "2.2uF" V 3389 4000 50  0000 C CNN
 F 2 "motor_drive_footprints:C_0603_1608Metric" H 3588 3850 50  0001 C CNN
 F 3 "~" H 3550 4000 50  0001 C CNN
@@
 	3550 3850 3400 3850
 Connection ~ 3550 3850
+$Comp
+L motor_drive:C C13
+U 1 1 5E5D273D
+P 4100 4000
+F 0 "C13" V 3848 4000 50  0000 C CNN
+F 1 "0.01uF" V 3939 4000 50  0000 C CNN
+F 2 "motor_drive_footprints:C_0603_1608Metric" H 4138 3850 50  0001 C CNN
+F 3 "~" H 4100 4000 50  0001 C CNN
+	1    4100 4000
+	1    0    0    -1
+$EndComp
 $EndSCHEMATC

Commit message: started layout
Parts:
- renumbered C12 to C21, C13 to C22
Changed lines of the file:
@@
 $Descr A4 11693 8268
 encoding utf-8
-Sheet 10 14
+Sheet 10 16
 Title ""
 Date ""
@@
 	4450 4150 3550 4150
 $Comp
-L motor_drive:C C12
+L motor_drive:C C21
 U 1 1 5E374B8C
 P 3550 4000
-F 0 "C12" V 3298 4000 50  0000 C CNN
+F 0 "C21" V 3298 4000 50  0000 C CNN
 F 1 "2.2uF" V 3389 4000 50  0000 C CNN
 F 2 "motor_drive_footprints:C_0603_1608Metric" H 3588 3850 50  0001 C CNN
@@
 Connection ~ 3550 3850
 $Comp
-L motor_drive:C C13
+L motor_drive:C C22
 U 1 1 5E5D273D
 P 4100 4000
-F 0 "C13" V 3848 4000 50  0000 C CNN
+F 0 "C22" V 3848 4000 50  0000 C CNN
 F 1 "0.01uF" V 3939 4000 50  0000 C CNN
 F 2 "motor_drive_footprints:C_0603_1608Metric" H 4138 3850 50  0001 C CNN

Commit message: layout
Connections:
- net GND: now also C22.2
- net VDD: now also C22.1
Changed lines of the file:
@@
 VDD
 NoConn ~ 4450 4050
-Wire Wire Line
-	4450 4150 3550 4150
 $Comp
 L motor_drive:C C21
@@
 $EndComp
 Wire Wire Line
-	4450 3850 3550 3850
-Wire Wire Line
 	3550 3850 3400 3850
-Connection ~ 3550 3850
 $Comp
 L motor_drive:C C22
@@
 	1    0    0    -1
 $EndComp
+Wire Wire Line
+	3550 3850 4100 3850
+Connection ~ 3550 3850
+Connection ~ 4100 3850
+Wire Wire Line
+	4100 3850 4450 3850
+Wire Wire Line
+	3550 4150 4100 4150
+Connection ~ 3550 4150
+Connection ~ 4100 4150
+Wire Wire Line
+	4100 4150 4450 4150
 $EndSCHEMATC

Commit message: second try at layout
Parts:
- renumbered C21 to C1, C22 to C2, U5 to U1
Changed lines of the file:
@@
 $Descr A4 11693 8268
 encoding utf-8
-Sheet 10 6
+Sheet 2 6
 Title ""
 Date ""
@@
 $EndDescr
 $Comp
-L motor_drive:ADA4571WHRZ-R7 U5
+L motor_drive:ADA4571WHRZ-R7 U1
 U 1 1 5E373274
 P 4450 3850
-F 0 "U5" H 5250 4237 60  0000 C CNN
+F 0 "U1" H 5250 4237 60  0000 C CNN
 F 1 "ADA4571WHRZ-R7" H 5250 4131 60  0000 C CNN
 F 2 "motor_drive_footprints:AD8418ABRMZ-RL" H 5250 4090 60  0001 C CNN
@@
 NoConn ~ 4450 4050
 $Comp
-L motor_drive:C C21
+L motor_drive:C C1
 U 1 1 5E374B8C
 P 3550 4000
-F 0 "C21" V 3298 4000 50  0000 C CNN
+F 0 "C1" V 3298 4000 50  0000 C CNN
 F 1 "2.2uF" V 3389 4000 50  0000 C CNN
 F 2 "motor_drive_footprints:C_0603_1608Metric" H 3588 3850 50  0001 C CNN
@@
 	3550 3850 3400 3850
 $Comp
-L motor_drive:C C22
+L motor_drive:C C2
 U 1 1 5E5D273D
 P 4100 4000
-F 0 "C22" V 3848 4000 50  0000 C CNN
+F 0 "C2" V 3848 4000 50  0000 C CNN
 F 1 "0.01uF" V 3939 4000 50  0000 C CNN
 F 2 "motor_drive_footprints:C_0603_1608Metric" H 4138 3850 50  0001 C CNN
