File: motor_drive_REV_1/F28027.sch (KiCad schematic (older format))
At the start: 15 parts

Commit message: organizing pinout and BOM
Parts:
- removed C?: C, symbol motor_drive:C
- removed R? (x5): R, symbol motor_drive:R
- added C25, C26, C33: 1uF, motor_drive_footprints:C_0603_1608Metric, symbol motor_drive:C
- added C28: 0.01uF, motor_drive_footprints:C_0603_1608Metric, symbol motor_drive:C
- added C32: 4.7uF, motor_drive_footprints:C_0603_1608Metric, symbol motor_drive:C
- added J3, J4: Conn_01x06, motor_drive_footprints:6pos_254, symbol Connector_Generic:Conn_01x06
- added L2: 2.2uF, motor_drive_footprints:C_0603_1608Metric, symbol motor_drive:L
- added R33, R34, R35, R36, R37, R38, R39, R40: 375, motor_drive_footprints:C_0603_1608Metric, symbol motor_drive:R
- added R41: R, motor_drive_footprints:C_0603_1608Metric, symbol motor_drive:R
- C24, C27: renamed from C?; value C -> 2.2uF; footprint (none) -> motor_drive_footprints:C_0603_1608Metric
- C29: renamed from C?; value C -> 4.7uF; footprint (none) -> motor_drive_footprints:C_0603_1608Metric
- C30: renamed from C?; value C -> 100pF; footprint (none) -> motor_drive_footprints:C_0603_1608Metric
- C31: renamed from C?; value C -> 1uF; footprint (none) -> motor_drive_footprints:C_0603_1608Metric
- L1: renamed from L?; value L -> 2.2uF; footprint (none) -> motor_drive_footprints:C_0603_1608Metric
- R31: renamed from R?; value R -> 2.2k; footprint (none) -> motor_drive_footprints:C_0603_1608Metric
- R32: renamed from R?; footprint (none) -> motor_drive_footprints:C_0603_1608Metric
- U8: renamed from U?; footprint PT48 -> motor_drive_footprints:TMS320F28027PTT
Connections:
- net labels added: GPIO_12, GPIO_32, GPIO_33, GPIO_34, GPIO_6, GPIO_7, JTAG_nTRST
- net labels removed: +5V, JTAG_nRESET, UART_RX_1, UART_TX_1
- wire segments 35 -> 67
Other:
- moved on the sheet: C24, C27, C29, C31, L1, R32

Commit message: piccolo pinout
Parts:
- added R? (x8): 375, motor_drive_footprints:C_0603_1608Metric, symbol motor_drive:R
- added U?: TMS20F28027PTT-custom, symbol motor_drive:TMS20F28027PTT-custom
Connections:
- net labels added: ADC_B7
- net labels removed: ADC_B5
- wire segments 67 -> 88
Other:
- moved on the sheet: C24, C25, C26, C27, C28, C29, C30, C31, C32, C33, J3, J4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

Commit message: working on adding thermistors but encountered too many hierarchicaly copies bug
Parts:
- removed C27: 2.2uF, motor_drive_footprints:C_0603_1608Metric, symbol motor_drive:C
- removed C28: 0.01uF, motor_drive_footprints:C_0603_1608Metric, symbol motor_drive:C
- removed R37, R38, R39, R40: 375, motor_drive_footprints:C_0603_1608Metric, symbol motor_drive:R
- removed U8: TMS320F28027PTT, motor_drive_footprints:TMS320F28027PTT, symbol motor_drive:TMS320F28027PTT
- added C23: 2.2uF, motor_drive_footprints:C_0603_1608Metric, symbol motor_drive:C
- added R27: 375, motor_drive_footprints:C_0603_1608Metric, symbol motor_drive:R
- added R29, R30, R31, R32: 10k, motor_drive_footprints:C_0603_1608Metric, symbol motor_drive:R
- C25, C26: value 1uF -> 0.01uF
- R26: renamed from R32; value R -> 4.7k
- R33, R34, R35, R36: value 375 -> 10k
- U8: renamed from U?; footprint (none) -> motor_drive_footprints:TMS320F28027PTT
- gave numbers to parts that had none: 8
- renumbered C32 to C27, C33 to C28, C30 to C29, C29 to C30, J3 to J5, J4 to J6, L2 to L1, L1 to L2, R41 to R25, R31 to R28
Connections:
- net labels added: PWM0, chip_reset
- net labels removed: PWM6
- wire segments 88 -> 85
- no-connect marks 2 -> 1
Other:
- moved on the sheet: C27, C28, C29, C30, C31, J5, J6, L1, L2, R25, R26, R28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

Commit message: started layout
Parts:
- renumbered C23 to C32, C24 to C33, C25 to C34, C26 to C35, C27 to C36, C28 to C37, C29 to C38, C30 to C39, C31 to C40, J5 to J4, J6 to J5, R25 to R23, R26 to R24, R27 to R25, R28 to R26, R29 to R27, R30 to R28, R31 to R29, R32 to R30, R33 to R31, R34 to R32, R35 to R33, R36 to R34, R37 to R35, R38 to R36, R39 to R37, R40 to R38, R41 to R39, R42 to R40, R43 to R41, R44 to R42
Changed lines of the file:
@@
 $Descr B 17000 11000
 encoding utf-8
-Sheet 13 14
+Sheet 13 16
 Title ""
 Date ""
@@
 $EndDescr
 $Comp
-L motor_drive:R R28
+L motor_drive:R R26
 U 1 1 5E2CBC65
 P 7000 6950
-F 0 "R28" H 7070 6996 50  0000 L CNN
+F 0 "R26" H 7070 6996 50  0000 L CNN
 F 1 "2.2k" H 7070 6905 50  0000 L CNN
 F 2 "motor_drive_footprints:C_0603_1608Metric" V 6930 6950 50  0001 C CNN
@@
 GND
 $Comp
-L motor_drive:C C31
+L motor_drive:C C40
 U 1 1 5E2D37BE
 P 8700 6750
-F 0 "C31" H 8815 6796 50  0000 L CNN
+F 0 "C40" H 8815 6796 50  0000 L CNN
 F 1 "1uF" H 8815 6705 50  0000 L CNN
 F 2 "motor_drive_footprints:C_0603_1608Metric" H 8738 6600 50  0001 C CNN
@@
 $EndComp
 $Comp
-L motor_drive:C C29
+L motor_drive:C C38
 U 1 1 5E2C88ED
 P 7000 7250
-F 0 "C29" H 7115 7296 50  0000 L CNN
+F 0 "C38" H 7115 7296 50  0000 L CNN
 F 1 "100pF" H 7115 7205 50  0000 L CNN
 F 2 "motor_drive_footprints:C_0603_1608Metric" H 7038 7100 50  0001 C CNN
@@
 $EndComp
 $Comp
-L motor_drive:C C30
+L motor_drive:C C39
 U 1 1 5E311B08
 P 8000 6750
-F 0 "C30" H 8115 6796 50  0000 L CNN
+F 0 "C39" H 8115 6796 50  0000 L CNN
 F 1 "4.7uF" H 8115 6705 50  0000 L CNN
 F 2 "motor_drive_footprints:C_0603_1608Metric" H 8038 6600 50  0001 C CNN
@@
 	8500 6400 8700 6400
 $Comp
-L motor_drive:R R26
+L motor_drive:R R24
 U 1 1 5E3169E2
 P 6550 3200
-F 0 "R26" H 6620 3246 50  0000 L CNN
+F 0 "R24" H 6620 3246 50  0000 L CNN
 F 1 "4.7k" H 6620 3155 50  0000 L CNN
 F 2 "motor_drive_footprints:C_0603_1608Metric" V 6480 3200 50  0001 C CNN
@@
 GPIO_7
 $Comp
-L Connector_Generic:Conn_01x06 J5
+L Connector_Generic:Conn_01x06 J4
 U 1 1 5E356D9E
 P 13100 5650
-F 0 "J5" H 13180 5642 50  0000 L CNN
+F 0 "J4" H 13180 5642 50  0000 L CNN
 F 1 "Conn_01x06" H 13180 5551 50  0000 L CNN
 F 2 "motor_drive_footprints:6pos_254" H 13100 5650 50  0001 C CNN
@@
 JTAG_nTRST
 $Comp
-L Connector_Generic:Conn_01x06 J6
+L Connector_Generic:Conn_01x06 J5
 U 1 1 5E35A7F5
 P 13100 6700
-F 0 "J6" H 13180 6692 50  0000 L CNN
+F 0 "J5" H 13180 6692 50  0000 L CNN
 F 1 "Conn_01x06" H 13180 6601 50  0000 L CNN
 F 2 "motor_drive_footprints:6pos_254" H 13100 6700 50  0001 C CNN
@@
 5.0V
 $Comp
-L motor_drive:R R25
+L motor_drive:R R23
 U 1 1 5E401F5C
 P 6450 8100
-F 0 "R25" H 6520 8146 50  0000 L CNN
+F 0 "R23" H 6520 8146 50  0000 L CNN
 F 1 "R" H 6520 8055 50  0000 L CNN
 F 2 "motor_drive_footprints:C_0603_1608Metric" V 6380 8100 50  0001 C CNN
@@
 	6450 8300 6450 8250
 $Comp
-L motor_drive:C C28
+L motor_drive:C C37
 U 1 1 5E3AB121
 P 6050 3000
-F 0 "C28" H 6165 3046 50  0000 L CNN
+F 0 "C37" H 6165 3046 50  0000 L CNN
 F 1 "1uF" H 6165 2955 50  0000 L CNN
 F 2 "motor_drive_footprints:C_0603_1608Metric" H 6088 2850 50  0001 C CNN
@@
 $EndComp
 $Comp
-L motor_drive:C C27
+L motor_drive:C C36
 U 1 1 5E3AB12E
 P 5350 3000
-F 0 "C27" H 5465 3046 50  0000 L CNN
+F 0 "C36" H 5465 3046 50  0000 L CNN
 F 1 "4.7uF" H 5465 2955 50  0000 L CNN
 F 2 "motor_drive_footprints:C_0603_1608Metric" H 5388 2850 50  0001 C CNN
@@
 SPI_CLK
 $Comp
-L motor_drive:R R41
+L motor_drive:R R39
 U 1 1 5E40175C
 P 11250 3500
-F 0 "R41" H 11320 3546 50  0000 L CNN
+F 0 "R39" H 11320 3546 50  0000 L CNN
 F 1 "375" H 11320 3455 50  0000 L CNN
 F 2 "motor_drive_footprints:C_0603_1608Metric" V 11180 3500 50  0001 C CNN
@@
 $EndComp
 $Comp
-L motor_drive:R R37
+L motor_drive:R R35
 U 1 1 5E401762
 P 10650 3300
-F 0 "R37" H 10720 3346 50  0000 L CNN
+F 0 "R35" H 10720 3346 50  0000 L CNN
 F 1 "375" H 10720 3255 50  0000 L CNN
 F 2 "motor_drive_footprints:C_0603_1608Metric" V 10580 3300 50  0001 C CNN
@@
 $EndComp
 $Comp
-L motor_drive:R R39
+L motor_drive:R R37
 U 1 1 5E401768
 P 10950 3400
-F 0 "R39" H 11020 3446 50  0000 L CNN
+F 0 "R37" H 11020 3446 50  0000 L CNN
 F 1 "375" H 11020 3355 50  0000 L CNN
 F 2 "motor_drive_footprints:C_0603_1608Metric" V 10880 3400 50  0001 C CNN
@@
 $EndComp
 $Comp
-L motor_drive:R R43
+L motor_drive:R R41
 U 1 1 5E40176E
 P 11550 3600
-F 0 "R43" H 11620 3646 50  0000 L CNN
+F 0 "R41" H 11620 3646 50  0000 L CNN
 F 1 "375" H 11620 3555 50  0000 L CNN
 F 2 "motor_drive_footprints:C_0603_1608Metric" V 11480 3600 50  0001 C CNN
@@
 JTAG_TDI
 $Comp
-L motor_drive:R R38
+L motor_drive:R R36
 U 1 1 5E4298D2
 P 10650 4550
-F 0 "R38" H 10720 4596 50  0000 L CNN
+F 0 "R36" H 10720 4596 50  0000 L CNN
 F 1 "375" H 10720 4505 50  0000 L CNN
 F 2 "motor_drive_footprints:C_0603_1608Metric" V 10580 4550 50  0001 C CNN
@@
 $EndComp
 $Comp
-L motor_drive:R R40
+L motor_drive:R R38
 U 1 1 5E4298D8
 P 10950 4650
-F 0 "R40" H 11020 4696 50  0000 L CNN
+F 0 "R38" H 11020 4696 50  0000 L CNN
 F 1 "375" H 11020 4605 50  0000 L CNN
 F 2 "motor_drive_footprints:C_0603_1608Metric" V 10880 4650 50  0001 C CNN
@@
 $EndComp
 $Comp
-L motor_drive:R R42
+L motor_drive:R R40
 U 1 1 5E4298DE
 P 11250 4750
-F 0 "R42" H 11320 4796 50  0000 L CNN
+F 0 "R40" H 11320 4796 50  0000 L CNN
 F 1 "375" H 11320 4705 50  0000 L CNN
 F 2 "motor_drive_footprints:C_0603_1608Metric" V 11180 4750 50  0001 C CNN
@@
 $EndComp
 $Comp
-L motor_drive:R R44
+L motor_drive:R R42
 U 1 1 5E4298E4
 P 11550 4850
-F 0 "R44" H 11620 4896 50  0000 L CNN
+F 0 "R42" H 11620 4896 50  0000 L CNN
 F 1 "375" H 11620 4805 50  0000 L CNN
 F 2 "motor_drive_footprints:C_0603_1608Metric" V 11480 4850 50  0001 C CNN
@@
 	6550 3350 6550 3850
 $Comp
-L motor_drive:R R27
+L motor_drive:R R25
 U 1 1 5E4297B3
 P 6800 7850
-F 0 "R27" H 6870 7896 50  0000 L CNN
+F 0 "R25" H 6870 7896 50  0000 L CNN
 F 1 "375" H 6870 7805 50  0000 L CNN
 F 2 "motor_drive_footprints:C_0603_1608Metric" V 6730 7850 50  0001 C CNN
@@
 5.0V
 $Comp
-L motor_drive:C C25
+L motor_drive:C C34
 U 1 1 5E499E4F
 P 4600 4350
-F 0 "C25" H 4715 4396 50  0000 L CNN
+F 0 "C34" H 4715 4396 50  0000 L CNN
 F 1 "0.01uF" H 4715 4305 50  0000 L CNN
 F 2 "motor_drive_footprints:C_0603_1608Metric" H 4638 4200 50  0001 C CNN
@@
 $EndComp
 $Comp
-L motor_drive:C C23
+L motor_drive:C C32
 U 1 1 5E499E55
 P 4050 4350
-F 0 "C23" H 4165 4396 50  0000 L CNN
+F 0 "C32" H 4165 4396 50  0000 L CNN
 F 1 "2.2uF" H 4165 4305 50  0000 L CNN
 F 2 "motor_drive_footprints:C_0603_1608Metric" H 4088 4200 50  0001 C CNN
@@
 5.0V
 $Comp
-L motor_drive:C C26
+L motor_drive:C C35
 U 1 1 5E4D3554
 P 4600 5550
-F 0 "C26" H 4715 5596 50  0000 L CNN
+F 0 "C35" H 4715 5596 50  0000 L CNN
 F 1 "0.01uF" H 4715 5505 50  0000 L CNN
 F 2 "motor_drive_footprints:C_0603_1608Metric" H 4638 5400 50  0001 C CNN
@@
 $EndComp
 $Comp
-L motor_drive:C C24
+L motor_drive:C C33
 U 1 1 5E4D355A
 P 4050 5550
-F 0 "C24" H 4165 5596 50  0000 L CNN
+F 0 "C33" H 4165 5596 50  0000 L CNN
 F 1 "2.2uF" H 4165 5505 50  0000 L CNN
 F 2 "motor_drive_footprints:C_0603_1608Metric" H 4088 5400 50  0001 C CNN
@@
 Connection ~ 6450 7850
 $Comp
-L motor_drive:R R30
+L motor_drive:R R28
 U 1 1 5E511168
 P 8600 4200
-F 0 "R30" H 8670 4246 50  0000 L CNN
+F 0 "R28" H 8670 4246 50  0000 L CNN
 F 1 "10k" H 8670 4155 50  0000 L CNN
 F 2 "motor_drive_footprints:C_0603_1608Metric" V 8530 4200 50  0001 C CNN
@@
 	7250 3300 9650 3300
 $Comp
-L motor_drive:R R32
+L motor_drive:R R30
 U 1 1 5E53E15B
 P 8950 4200
-F 0 "R32" H 9020 4246 50  0000 L CNN
+F 0 "R30" H 9020 4246 50  0000 L CNN
 F 1 "10k" H 9020 4155 50  0000 L CNN
 F 2 "motor_drive_footprints:C_0603_1608Metric" V 8880 4200 50  0001 C CNN
@@
 $EndComp
 $Comp
-L motor_drive:R R34
+L motor_drive:R R32
 U 1 1 5E54172F
 P 9300 4200
-F 0 "R34" H 9370 4246 50  0000 L CNN
+F 0 "R32" H 9370 4246 50  0000 L CNN
 F 1 "10k" H 9370 4155 50  0000 L CNN
 F 2 "motor_drive_footprints:C_0603_1608Metric" V 9230 4200 50  0001 C CNN
@@
 $EndComp
 $Comp
-L motor_drive:R R36
+L motor_drive:R R34
 U 1 1 5E544D62
 P 9650 4200
-F 0 "R36" H 9720 4246 50  0000 L CNN
+F 0 "R34" H 9720 4246 50  0000 L CNN
 F 1 "10k" H 9720 4155 50  0000 L CNN
 F 2 "motor_drive_footprints:C_0603_1608Metric" V 9580 4200 50  0001 C CNN
@@
 $EndComp
 $Comp
-L motor_drive:R R29
+L motor_drive:R R27
 U 1 1 5E549B17
 P 8600 2950
-F 0 "R29" H 8670 2996 50  0000 L CNN
+F 0 "R27" H 8670 2996 50  0000 L CNN
 F 1 "10k" H 8670 2905 50  0000 L CNN
 F 2 "motor_drive_footprints:C_0603_1608Metric" V 8530 2950 50  0001 C CNN
@@
 $EndComp
 $Comp
-L motor_drive:R R31
+L motor_drive:R R29
 U 1 1 5E549B1D
 P 8950 2950
-F 0 "R31" H 9020 2996 50  0000 L CNN
+F 0 "R29" H 9020 2996 50  0000 L CNN
 F 1 "10k" H 9020 2905 50  0000 L CNN
 F 2 "motor_drive_footprints:C_0603_1608Metric" V 8880 2950 50  0001 C CNN
@@
 $EndComp
 $Comp
-L motor_drive:R R33
+L motor_drive:R R31
 U 1 1 5E549B23
 P 9300 2950
-F 0 "R33" H 9370 2996 50  0000 L CNN
+F 0 "R31" H 9370 2996 50  0000 L CNN
 F 1 "10k" H 9370 2905 50  0000 L CNN
 F 2 "motor_drive_footprints:C_0603_1608Metric" V 9230 2950 50  0001 C CNN
@@
 $EndComp
 $Comp
-L motor_drive:R R35
+L motor_drive:R R33
 U 1 1 5E549B29
 P 9650 2950
-F 0 "R35" H 9720 2996 50  0000 L CNN
+F 0 "R33" H 9720 2996 50  0000 L CNN
 F 1 "10k" H 9720 2905 50  0000 L CNN
 F 2 "motor_drive_footprints:C_0603_1608Metric" V 9580 2950 50  0001 C CNN

Commit message: layout
Connections:
- net SPI_MISO: now also J4.2 (Pin_2); no longer J4.1 (Pin_1)
- net SPI_MOSI: now also J4.1 (Pin_1); no longer J4.2 (Pin_2)
Changed lines of the file:
@@
 GND
 Text Label 12450 5450 0    50   ~ 0
+SPI_MOSI
+Text Label 12450 5550 0    50   ~ 0
 SPI_MISO
-Text Label 12450 5550 0    50   ~ 0
-SPI_MOSI
 Text Label 12450 5650 0    50   ~ 0
 SPI_CLK

Commit message: gate drive rework and schematic re-organization
Parts:
- added D? (x6): LED, symbol motor_drive:LED
- added R? (x8): 10k, motor_drive_footprints:C_0603_1608Metric, symbol motor_drive:R
- added SW? (x2): SW_Push, symbol motor_drive:SW_Push
- R20: renamed from R23; value R -> 4.7k
- renumbered C32 to C27, C33 to C28, C34 to C29, C35 to C30, C36 to C31, C37 to C32, C38 to C33, C39 to C34, C40 to C35, R24 to R21, R25 to R22, R26 to R23, R27 to R24, R28 to R25, R29 to R26, R30 to R27, R31 to R28, R32 to R29, R33 to R30, R34 to R31, R35 to R32, R36 to R33, R37 to R34, R38 to R35, R39 to R36, R40 to R37, R41 to R38, R42 to R39, U8 to U7
Connections:
- net 5.0V: now also D?.2 (A), D?.2 (A), D?.2 (A), D?.2 (A), D?.2 (A), D?.2 (A), R?.1, R?.1
- net GND: now also SW?.2, SW?.2
- net GPIO_32 renamed LED_0
- net LED_0: now also R?.2
- net GPIO_33 renamed LED_1
- net LED_1: now also R?.2
- net GPIO_34 renamed LED_2
- net LED_2: now also R?.2
- net GPIO_6 renamed BUTTON_0
- net BUTTON_0: now also R?.2, SW?.1
- net GPIO_7 renamed BUTTON_1
- net BUTTON_1: now also R?.2, SW?.1
- net PWM0 renamed PWM_0
- net PWM1 renamed PWM_1
- net PWM2 renamed PWM_2
- net PWM3 renamed LED_3
- net LED_3: now also R?.2
- net PWM4 renamed LED_4
- net LED_4: now also R?.2
- net PWM5 renamed LED_5
- net LED_5: now also R?.2
- new net: D?.1 (K), R?.1 (x6)

Commit message: second try at layout
Parts:
- removed SW? (x2): SW_Push, symbol motor_drive:SW_Push
- added SW1, SW2: EVQ-Q2B01W, motor_drive_footprints:EVQ-Q2B01W, symbol motor_drive:EVQ-Q2B01W
- D1, D2, D3, D4, D5, D6: renamed from D?; footprint (none) -> motor_drive_footprints:C_0603_1608Metric
- gave numbers to parts that had none: 8
- renumbered C30 to C10, C31 to C11, C32 to C12, C33 to C13, C34 to C14, C35 to C15, C27 to C7, C28 to C8, C29 to C9, J4 to J2, J5 to J3, R20 to R19, R21 to R20, R22 to R21, R23 to R22, R24 to R23, R25 to R24, R26 to R25, R27 to R26, R28 to R27, R29 to R28, R30 to R29, R31 to R30, R32 to R31, R33 to R32, R34 to R33, R35 to R34, R36 to R35, R37 to R36, R38 to R37, R39 to R38, U7 to U3
Connections:
- net BUTTON_0: now also SW1.1
- net BUTTON_1: now also SW2.1
- net GND: now also SW1.4, SW2.4
Other:
- moved on the sheet: R12
