File: motor_drive_REV_1/MAIN.sch (KiCad schematic (older format))
At the start: 11 parts

Commit message: work on component libraries and schematic
Parts:
- removed C?: C, symbol Device:C
- removed M? (x2): Conn_01x01, symbol Connector_Generic:Conn_01x01
- removed R?: R, symbol Device:R
- removed U?: TJA1051TK-3, Package_DFN_QFN:DFN-8-1EP_3x3mm_P0.65mm_EP1.55x2.4mm, symbol Interface_CAN_LIN:TJA1051TK-3
- removed U?: DRV8301, symbol motor_drive:DRV8301
- removed U?: ADM4853WARZ-RL7, R_8, symbol ADM4853:ADM4853WARZ-RL7
- removed U?: SN65LBC176QDRQ1, D8, symbol SN65LB:SN65LBC176QDRQ1
Connections:
- net labels added: A, B, DC_neg, DC_pos, IDC_sense_n, IDC_sense_p, VDC_sense_n, VDC_sense_p
- net labels removed: 5.0V, DC+, GND, I_sense_2, I_sense_3, VCC, V_sense_1, V_sense_1n, V_sense_1p, V_sense_2, V_sense_2n, V_sense_2p, V_sense_3, V_sense_3n, V_sense_3p
- wire segments 65 -> 20

Commit message: organizing pinout and BOM
Parts:
- removed M? (x3): Conn_01x01, symbol Connector_Generic:Conn_01x01
- added J1: Conn_01x02, motor_drive_footprints:2pos_254, symbol Connector_Generic:Conn_01x02
- added J2: Conn_01x03, motor_drive_footprints:3pos_254, symbol Connector_Generic:Conn_01x03
Connections:
- net labels added: 5.0V, BUTTON_0, BUTTON_1, CLK, DEnRE, GH_1, GH_2, GH_3, GL_1, GL_2, GL_3, GND, HS_1, HS_2, HS_3, IDC_sense, I_sense_2, I_sense_3, I_sense_n1, I_sense_n2, I_sense_n3, I_sense_p1, I_sense_p2, I_sense_p3, LED_0, LED_1, LED_2, LS_1, LS_2, LS_3, MISO, MOSI, SW_1, SW_2, SW_3, UART_RX, UART_TX, VDC_sense, balance, cos, nEN, sin
- wire segments 20 -> 69

Commit message: piccolo pinout
Changed lines of the file:
@@
 F11 "ADC_B3" I R 7500 6600 50
 F12 "ADC_B4" I R 7500 6750 50
-F13 "ADC_B5" I R 7500 6900 50
-F14 "ADC_B6" I R 7500 7050 50
-F15 "PWM1" I R 7500 3800 50
-F16 "PWM2" I R 7500 3950 50
-F17 "PWM3" I R 7500 4100 50
-F18 "PWM4" I R 7500 4250 50
-F19 "PWM5" I R 7500 4400 50
-F20 "PWM6" I R 7500 4550 50
-F21 "SPI_MOSI" I L 5650 3800 50
-F22 "SPI_MISO" I L 5650 3950 50
-F23 "SPI_CLK" I L 5650 4100 50
-F24 "5.0V" I L 5650 6900 50
-F25 "GND" I L 5650 7050 50
-F26 "SPI_nENABLE" I L 5650 4250 50
-F27 "UART_TX" I L 5650 4950 50
-F28 "UART_RX" I L 5650 5100 50
-F29 "GPIO_34" I L 5650 5650 50
-F30 "GPIO_33" I L 5650 5800 50
-F31 "GPIO_32" I L 5650 5950 50
-F32 "GPIO_6" I L 5650 6400 50
-F33 "GPIO_12" I L 5650 6100 50
-F34 "GPIO_7" I L 5650 6250 50
+F13 "ADC_B6" I R 7500 6900 50
+F14 "PWM1" I R 7500 3800 50
+F15 "PWM2" I R 7500 3950 50
+F16 "PWM3" I R 7500 4100 50
+F17 "PWM4" I R 7500 4250 50
+F18 "PWM5" I R 7500 4400 50
+F19 "PWM6" I R 7500 4550 50
+F20 "5.0V" I L 5650 6900 50
+F21 "GND" I L 5650 7050 50
+F22 "UART_TX" I L 5650 4950 50
+F23 "UART_RX" I L 5650 5100 50
+F24 "GPIO_34" I L 5650 5650 50
+F25 "GPIO_33" I L 5650 5800 50
+F26 "GPIO_32" I L 5650 5950 50
+F27 "GPIO_6" I L 5650 6400 50
+F28 "GPIO_12" I L 5650 6100 50
+F29 "GPIO_7" I L 5650 6250 50
+F30 "ADC_B7" I R 7500 7050 50
 $EndSheet
 Text Label 5250 6100 0    50   ~ 0

Commit message: working on adding thermistors but encountered too many hierarchicaly copies bug
Parts:
- renumbered J2 to J4
Connections:
- net labels added: chip_reset, therm_1, therm_2
- wire segments 69 -> 70
Changed lines of the file:
@@
 I_sense_2
 Text Label 7500 6600 0    50   ~ 0
-IDC_sense
+therm_1
 Text Label 7500 6750 0    50   ~ 0
-VDC_sense
+therm_2
 Text Label 7500 6900 0    50   ~ 0
 sin
-Text Label 5450 3800 0    50   ~ 0
+Text Label 5450 4050 0    50   ~ 0
 MOSI
-Text Label 5450 3950 0    50   ~ 0
+Text Label 5450 4200 0    50   ~ 0
 MISO
-Text Label 5450 4100 0    50   ~ 0
+Text Label 5450 4350 0    50   ~ 0
 CLK
-Text Label 5450 4250 0    50   ~ 0
+Text Label 5450 4500 0    50   ~ 0
 nEN
 Wire Wire Line
-	5450 3800 5650 3800
-Wire Wire Line
-	5450 3950 5650 3950
-Wire Wire Line
-	5450 4100 5650 4100
-Wire Wire Line
-	5450 4250 5650 4250
+	5450 4050 5650 4050
+Wire Wire Line
+	5450 4200 5650 4200
+Wire Wire Line
+	5450 4350 5650 4350
+Wire Wire Line
+	5450 4500 5650 4500
 Text Label 5450 6900 0    50   ~ 0
 5.0V
@@
 F12 "ADC_B4" I R 7500 6750 50
 F13 "ADC_B6" I R 7500 6900 50
-F14 "PWM1" I R 7500 3800 50
-F15 "PWM2" I R 7500 3950 50
-F16 "PWM3" I R 7500 4100 50
-F17 "PWM4" I R 7500 4250 50
-F18 "PWM5" I R 7500 4400 50
-F19 "PWM6" I R 7500 4550 50
-F20 "5.0V" I L 5650 6900 50
-F21 "GND" I L 5650 7050 50
-F22 "UART_TX" I L 5650 4950 50
-F23 "UART_RX" I L 5650 5100 50
-F24 "GPIO_34" I L 5650 5650 50
-F25 "GPIO_33" I L 5650 5800 50
-F26 "GPIO_32" I L 5650 5950 50
-F27 "GPIO_6" I L 5650 6400 50
-F28 "GPIO_12" I L 5650 6100 50
-F29 "GPIO_7" I L 5650 6250 50
-F30 "ADC_B7" I R 7500 7050 50
+F14 "PWM1" I R 7500 3950 50
+F15 "PWM2" I R 7500 4100 50
+F16 "PWM3" I R 7500 4250 50
+F17 "PWM4" I R 7500 4400 50
+F18 "PWM5" I R 7500 4550 50
+F19 "5.0V" I L 5650 6900 50
+F20 "GND" I L 5650 7050 50
+F21 "UART_TX" I L 5650 4950 50
+F22 "UART_RX" I L 5650 5100 50
+F23 "GPIO_34" I L 5650 5650 50
+F24 "GPIO_33" I L 5650 5800 50
+F25 "GPIO_32" I L 5650 5950 50
+F26 "GPIO_6" I L 5650 6400 50
+F27 "GPIO_12" I L 5650 6100 50
+F28 "GPIO_7" I L 5650 6250 50
+F29 "ADC_B7" I R 7500 7050 50
+F30 "PWM0" I R 7500 3800 50
+F31 "chip_reset" I L 5650 3650 50
+F32 "SPI_MISO" I L 5650 4200 50
+F33 "SPI_MOSI" I L 5650 4050 50
+F34 "SPI_nENABLE" I L 5650 4350 50
+F35 "SPI_CLK" I L 5650 4500 50
 $EndSheet
 Text Label 5250 6100 0    50   ~ 0
@@
 	5250 6400 5650 6400
 $Comp
-L Connector_Generic:Conn_01x03 J2
+L Connector_Generic:Conn_01x03 J4
 U 1 1 5E32DF06
 P 16050 3500
-F 0 "J2" H 16130 3542 50  0000 L CNN
+F 0 "J4" H 16130 3542 50  0000 L CNN
 F 1 "Conn_01x03" H 16130 3451 50  0000 L CNN
 F 2 "motor_drive_footprints:3pos_254" H 16050 3500 50  0001 C CNN
@@
 Wire Wire Line
 	1800 5800 2000 5800
+Text Label 5250 3650 0    50   ~ 0
+chip_reset
+Wire Wire Line
+	5250 3650 5650 3650
 $EndSCHEMATC

Commit message: started layout
Parts:
- removed J4: Conn_01x03, motor_drive_footprints:3pos_254, symbol Connector_Generic:Conn_01x03
- added J1: Conn_01x04, motor_drive_footprints:4pos_254, symbol Connector_Generic:Conn_01x04
- added J3: Conn_01x04, motor_drive_footprints:4pos_338, symbol Connector_Generic:Conn_01x04
- renumbered J1 to J2
Connections:
- net DC_Link_Input/DC_pos_in is gone; now on net IDC_sense_p: J2.2 (Pin_2)
- net A: now also J1.4 (Pin_4)
- net B: now also J1.3 (Pin_3)
- net GND: now also J1.1 (Pin_1)
- net balance: now also J1.2 (Pin_2)
- net half_bridge_1/M: now also J3.1 (Pin_1)
- net half_bridge_2/M: now also J3.2 (Pin_2)
- net half_bridge_3/M: now also J3.3 (Pin_3)
- new net phase_shield: J3.4 (Pin_4)
Other:
- moved on the sheet: J2

Commit message: layout
Changed lines of the file:
@@
 $EndSheet
 Text Label 9400 4800 0    50   ~ 0
-I_sense_1n
+I_sense_n1
 Text Label 9400 4650 0    50   ~ 0
-I_sense_1p
+I_sense_p1
 Text Label 9400 5750 0    50   ~ 0
-I_sense_2n
+I_sense_n2
 Text Label 9400 5600 0    50   ~ 0
-I_sense_2p
+I_sense_p2
 Text Label 9400 6700 0    50   ~ 0
-I_sense_3n
+I_sense_n3
 Text Label 9400 6550 0    50   ~ 0
-I_sense_3p
+I_sense_p3
 Text Label 10600 5200 0    50   ~ 0
 5.0V

Commit message: gate drive rework and schematic re-organization
Parts:
- removed J1: Conn_01x04, motor_drive_footprints:4pos_254, symbol Connector_Generic:Conn_01x04
- removed J2: Conn_01x02, motor_drive_footprints:2pos_254, symbol Connector_Generic:Conn_01x02
- removed J3: Conn_01x04, motor_drive_footprints:4pos_338, symbol Connector_Generic:Conn_01x04

Commit message: second try at layout
Connections:
- no-connect marks 0 -> 3
Changed lines of the file:
@@
 $EndDescr
 $Sheet
-S 4500 4000 900  1000
+S 5000 3500 900  1000
 U 5E373134
 F0 "Position sensor" 50
 F1 "ADA4571WHRZ.sch" 50
-F2 "GND" I R 5400 4800 50
-F3 "SIN" I R 5400 4200 50
-F4 "COS" I R 5400 4350 50
-F5 "VDD" I R 5400 4650 50
+F2 "GND" I R 5900 4300 50
+F3 "SIN" I R 5900 3700 50
+F4 "COS" I R 5900 3850 50
+F5 "VDD" I R 5900 4150 50
 $EndSheet
 $Sheet
-S 4500 2000 950  1150
+S 5000 1500 950  1150
 U 5E38D632
 F0 "RS422" 50
 F1 "SN65.sch" 50
-F2 "GND" I R 5450 2950 50
-F3 "VCC" I R 5450 2800 50
-F4 "D" I R 5450 2350 50
-F5 "R" I R 5450 2500 50
-F6 "DEnRE" I R 5450 2200 50
+F2 "GND" I R 5950 2450 50
+F3 "VCC" I R 5950 2300 50
+F4 "D" I R 5950 1850 50
+F5 "R" I R 5950 2000 50
+F6 "DEnRE" I R 5950 1700 50
 $EndSheet
-Text Label 5400 4200 0    50   ~ 0
+Text Label 5900 3700 0    50   ~ 0
 sin
-Text Label 5400 4350 0    50   ~ 0
+Text Label 5900 3850 0    50   ~ 0
 cos
-Text Label 5400 4650 0    50   ~ 0
+Text Label 5900 4150 0    50   ~ 0
 5.0V
-Text Label 5400 4800 0    50   ~ 0
+Text Label 5900 4300 0    50   ~ 0
 GND
-Text Label 8850 3000 0    50   ~ 0
+Text Label 9350 2500 0    50   ~ 0
 I_sense_2
-Text Label 8850 3150 0    50   ~ 0
-I_sense_3
-Text Label 8850 3300 0    50   ~ 0
+Text Label 9350 2650 0    50   ~ 0
 sin
-Text Label 8850 3450 0    50   ~ 0
+Text Label 9350 2800 0    50   ~ 0
 cos
-Text Label 8850 4100 0    50   ~ 0
+Text Label 9350 3600 0    50   ~ 0
 I_sense_1
-Text Label 8850 4250 0    50   ~ 0
+Text Label 9350 3750 0    50   ~ 0
 I_sense_2
-Text Label 8850 4400 0    50   ~ 0
+Text Label 9350 3900 0    50   ~ 0
 therm_1
-Text Label 8850 4550 0    50   ~ 0
+Text Label 9350 4050 0    50   ~ 0
 therm_2
-Text Label 8850 4700 0    50   ~ 0
+Text Label 9350 4200 0    50   ~ 0
 sin
-Text Label 6800 2600 0    50   ~ 0
+Text Label 7300 2100 0    50   ~ 0
 MOSI
-Text Label 6800 2750 0    50   ~ 0
+Text Label 7300 2250 0    50   ~ 0
 MISO
-Text Label 6800 2900 0    50   ~ 0
+Text Label 7300 2400 0    50   ~ 0
 CLK
-Text Label 6800 3050 0    50   ~ 0
+Text Label 7300 2550 0    50   ~ 0
 nEN
 Wire Wire Line
-	6800 2600 7000 2600
+	7300 2100 7500 2100
 Wire Wire Line
-	6800 2750 7000 2750
+	7300 2250 7500 2250
 Wire Wire Line
-	6800 2900 7000 2900
+	7300 2400 7500 2400
 Wire Wire Line
-	6800 3050 7000 3050
-Text Label 6800 4700 0    50   ~ 0
+	7300 2550 7500 2550
+Text Label 7300 4200 0    50   ~ 0
 5.0V
-Text Label 6800 4850 0    50   ~ 0
+Text Label 7300 4350 0    50   ~ 0
 GND
 Wire Wire Line
-	6800 4850 7000 4850
+	7300 4350 7500 4350
 Wire Wire Line
-	6800 4700 7000 4700
-Text Label 5450 2800 0    50   ~ 0
+	7300 4200 7500 4200
+Text Label 5950 2300 0    50   ~ 0
 5.0V
-Text Label 5450 2950 0    50   ~ 0
+Text Label 5950 2450 0    50   ~ 0
 GND
-Text Label 5450 2350 0    50   ~ 0
+Text Label 5950 1850 0    50   ~ 0
 UART_TX
-Text Label 5450 2500 0    50   ~ 0
+Text Label 5950 2000 0    50   ~ 0
 UART_RX
-Text Label 5450 2200 0    50   ~ 0
+Text Label 5950 1700 0    50   ~ 0
 DEnRE
 $Sheet
-S 7000 2000 1850 3050
+S 7500 1500 1850 3050
 U 5E2C4A87
 F0 "F28027" 50
 F1 "F28027.sch" 50
-F2 "ADC_A0" I R 8850 2850 50
-F3 "ADC_A1" I R 8850 3000 50
-F4 "ADC_A2" I R 8850 3150 50
-F5 "ADC_A3" I R 8850 3300 50
-F6 "ADC_A4" I R 8850 3450 50
-F7 "ADC_A6" I R 8850 3600 50
-F8 "ADC_A7" I R 8850 3750 50
-F9 "ADC_B1" I R 8850 4100 50
-F10 "ADC_B2" I R 8850 4250 50
-F11 "ADC_B3" I R 8850 4400 50
-F12 "ADC_B4" I R 8850 4550 50
-F13 "ADC_B6" I R 8850 4700 50
-F14 "PWM1" I R 8850 2350 50
-F15 "PWM2" I R 8850 2500 50
-F19 "5.0V" I L 7000 4700 50
-F20 "GND" I L 7000 4850 50
-F21 "UART_TX" I L 7000 3500 50
-F22 "UART_RX" I L 7000 3650 50
-F27 "GPIO_12" I L 7000 3800 50
-F29 "ADC_B7" I R 8850 4850 50
-F30 "PWM0" I R 8850 2200 50
-F31 "chip_reset" I L 7000 2200 50
-F32 "SPI_MISO" I L 7000 2750 50
-F33 "SPI_MOSI" I L 7000 2600 50
-F34 "SPI_nENABLE" I L 7000 2900 50
-F35 "SPI_CLK" I L 7000 3050 50
+F2 "ADC_A0" I R 9350 2350 50
+F3 "ADC_A1" I R 9350 2500 50
+F4 "ADC_A2" I R 9350 2650 50
+F5 "ADC_A3" I R 9350 2800 50
+F6 "ADC_A4" I R 9350 2950 50
+F7 "ADC_A6" I R 9350 3100 50
+F8 "ADC_A7" I R 9350 3250 50
+F9 "ADC_B1" I R 9350 3600 50
+F10 "ADC_B2" I R 9350 3750 50
+F11 "ADC_B3" I R 9350 3900 50
+F12 "ADC_B4" I R 9350 4050 50
+F13 "ADC_B6" I R 9350 4200 50
+F14 "PWM1" I R 9350 1850 50
+F15 "PWM2" I R 9350 2000 50
+F16 "5.0V" I L 7500 4200 50
+F17 "GND" I L 7500 4350 50
+F18 "UART_TX" I L 7500 3000 50
+F19 "UART_RX" I L 7500 3150 50
+F20 "GPIO_12" I L 7500 3300 50
+F21 "ADC_B7" I R 9350 4350 50
+F22 "PWM0" I R 9350 1700 50
+F23 "chip_reset" I L 7500 1700 50
+F24 "SPI_MISO" I L 7500 2250 50
+F25 "SPI_MOSI" I L 7500 2100 50
+F26 "SPI_nENABLE" I L 7500 2400 50
+F27 "SPI_CLK" I L 7500 2550 50
 $EndSheet
-Text Label 6600 3800 0    50   ~ 0
+Text Label 7100 3300 0    50   ~ 0
 DEnRE
-Text Label 8850 4850 0    50   ~ 0
+Text Label 9350 4350 0    50   ~ 0
 cos
-Text Label 6650 3500 0    50   ~ 0
+Text Label 7150 3000 0    50   ~ 0
 UART_TX
-Text Label 6650 3650 0    50   ~ 0
+Text Label 7150 3150 0    50   ~ 0
 UART_RX
 Wire Wire Line
-	6650 3500 7000 3500
+	7150 3000 7500 3000
 Wire Wire Line
-	6650 3650 7000 3650
+	7150 3150 7500 3150
 Wire Wire Line
-	6600 3800 7000 3800
-Text Label 8850 2850 0    50   ~ 0
+	7100 3300 7500 3300
+Text Label 9350 2350 0    50   ~ 0
 I_sense_1
-Text Label 6600 2200 0    50   ~ 0
+Text Label 7100 1700 0    50   ~ 0
 chip_reset
 Wire Wire Line
-	6600 2200 7000 2200
+	7100 1700 7500 1700
 $Sheet
-S 10050 2000 850  1900
+S 10550 1500 900  1700
 U 5E524F16
 F0 "power" 50
 F1 "power_stage.sch" 50
-F2 "PWM_1" I L 10050 2300 50
-F3 "GND" I L 10050 3000 50
-F4 "VDD" I L 10050 2850 50
-F5 "PWM_0" I L 10050 2150 50
-F6 "PWM_2" I L 10050 2450 50
-F7 "I_sense_0" I L 10050 3300 50
-F8 "I_sense_1" I L 10050 3450 50
-F9 "I_sense_2" I L 10050 3600 50
+F2 "PWM_1" I L 10550 1850 50
+F3 "GND" I L 10550 2500 50
+F4 "VDD" I L 10550 2350 50
+F5 "PWM_0" I L 10550 1700 50
+F6 "PWM_2" I L 10550 2000 50
+F7 "I_sense_0" I L 10550 2800 50
+F8 "I_sense_1" I L 10550 2950 50
 $EndSheet
 $Sheet
-S 10050 4150 800  900
+S 10550 3650 800  900
 U 5E9C38D7
 F0 "temperature" 50
 F1 "thermistors.sch" 50
-F2 "therm_0" I L 10050 4300 50
-F3 "GND" I L 10050 4900 50
-F4 "therm_1" I L 10050 4450 50
-F5 "VCC" I L 10050 4750 50
+F2 "therm_0" I L 10550 3800 50
+F3 "GND" I L 10550 4400 50
+F4 "therm_1" I L 10550 3950 50
+F5 "VCC" I L 10550 4250 50
 $EndSheet
-Text Label 8850 2200 0    50   ~ 0
+Text Label 9350 1700 0    50   ~ 0
 PWM_0
-Text Label 8850 2350 0    50   ~ 0
+Text Label 9350 1850 0    50   ~ 0
 PWM_1
-Text Label 8850 2500 0    50   ~ 0
+Text Label 9350 2000 0    50   ~ 0
 PWM_2
+Text Label 10550 1700 2    50   ~ 0
+PWM_0
+Text Label 10550 1850 2    50   ~ 0
+PWM_1
+Text Label 10550 2000 2    50   ~ 0
+PWM_2
+Text Label 10550 2350 2    50   ~ 0
+7.5V
+Text Label 10550 2500 2    50   ~ 0
+GND
+Text Label 10550 2800 2    50   ~ 0
+I_sense_0
+Text Label 10550 2950 2    50   ~ 0
+I_sense_1
+Text Label 10550 3800 2    50   ~ 0
+therm_0
+Text Label 10550 3950 2    50   ~ 0
+therm_1
+Text Label 10550 4250 2    50   ~ 0
+5.0V
+Text Label 10550 4400 2    50   ~ 0
+GND
+NoConn ~ 9450 2950
+NoConn ~ 9450 3100
+NoConn ~ 9450 3250
+Wire Wire Line
+	9350 2950 9450 2950
+Wire Wire Line
+	9450 3100 9350 3100
+Wire Wire Line
+	9450 3250 9350 3250
 $EndSCHEMATC
