File: motor_drive_REV_1/power_stage.sch (KiCad schematic (older format))
At the start: 59 parts

Commit message: second try at layout
Parts:
- removed C?: 1uF, motor_drive_footprints:C_0603_1608Metric, symbol Device:C
- removed C?: 0.01uF, motor_drive_footprints:C_0603_1608Metric, symbol Device:C
- removed R?: WSL20101L000FEA18, motor_drive_footprints:WSL20101L000FEA18, symbol motor_drive:WSL20101L000FEA18
- removed U?: AD8418ABRMZ-RL, RM_8, symbol motor_drive:AD8418ABRMZ-RL
- C33, C34, C35, C36, C37, C38, C39, C40, C41: renamed from C?; footprint (none) -> motor_drive_footprints:C_0603_1608Metric
- J4: renamed from J?; footprint (none) -> motor_drive_footprints:3pos_254
- R39, R40, R41, R42: renamed from R?; footprint (none) -> motor_drive_footprints:C_0603_1608Metric
- U4, U5, U6: renamed from U?; footprint D8 -> motor_drive_footprints:TPS28225DR
- U7, U8: renamed from U?; footprint RM_8 -> motor_drive_footprints:AD8418ABRMZ-RL
- gave numbers to parts that had none: 36
Connections:
- net W is gone; now on net SW_2: J5.3 (Pin_3)
- net V: now also R49.1, U8.8 (+IN)
